File: kicad-pcb/RP2350_60QFN_minimal.kicad_pcb (KiCad board)
At the start: 2 copper layers, 54 x 85.6 mm, 517 parts, among them J1 USB_C_Receptacle_USB2.0_14P, J3 TP4057, Q6 HL-2302V, Q7 HL-2302V, U1 RP2350A, U2 REG_3.3V, U3 ZD25WQ32CEIGR, U4 LIS2DH12TR, U5 DW01A, Y1 ABM8-272-T3

Commit message: DrillSense business card adaptation
- Replace back silkscreen text: Nick Johnson -> Eric Datum, Embedded Design -> DRILLSENSE, contact info -> drillsense.com
- Fix critical pressure solver bug in fluid_sim_crate (line 1026: self.u -> self.v, += -> -=)
- Add DrillSense ≠ mark startup animation (3-second display before fluid sim starts)
Other:
- board text added: "DRILLSENSE"
- board text added: "Eric Datum"
- board text added: "eric@drillsense.com drillsense.com"
- board text removed: "Embedded Design"
- board text removed: "Nicholas-L-Johnson@pm.me GitHub.com/Nicholas-L-Johnson/flip-card"
- board text removed: "Nick Johnson"
Changed lines of the file:
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@@
 		(layer "Edge.Cuts")
 	)
-	(gr_text "Embedded Design"
+	(gr_text "DRILLSENSE"
 		(at 14.01 3.53 90)
 		(layer "B.SilkS")
@@
 			(justify left top mirror)
 		)
-		(render_cache "Embedded Design" 90
+		(render_cache "DRILLSENSE" 90
 			(polygon
 				(pts
@@
 		)
 	)
-	(gr_text "Nicholas-L-Johnson@pm.me\nGitHub.com/Nicholas-L-Johnson/flip-card"
+	(gr_text "eric@drillsense.com\ndrillsense.com"
 		(at 42.47 3.84 90)
 		(layer "B.SilkS")
@@
 			(justify left top mirror)
 		)
-		(render_cache "Nicholas-L-Johnson@pm.me\nGitHub.com/Nicholas-L-Johnson/flip-card"
+		(render_cache "eric@drillsense.com\ndrillsense.com"
 			90
 			(polygon
@@
 		)
 	)
-	(gr_text "Nick Johnson"
+	(gr_text "Eric Datum"
 		(at 4.23 3.34 90)
 		(layer "B.SilkS")
@@
 			(justify left top mirror)
 		)
-		(render_cache "Nick Johnson" 90
-			(polygon
-				(pts
+		(render_cache "Eric Datum" 90
+			(polygon
+				(pts
